File: BTSTest/BTSTest.kicad_sch (KiCad schematic)
At the start: 72 parts, among them J1 197054001, J2 197054001, Q1 BC817, Q2 BC807, U1 BTS700121ESPXUMA1, U2 Pico, U3 TC1047VNBTR, U4 6mm_hole, U5 BTS70041EPPXUMA1, U6 INA219AxD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

Commit message: Update
Parts:
- C11, C9: value 10uF -> 1uF
Changed lines of the file:
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@@
       (effects (font (size 1.27 1.27)) (justify left))
     )
-    (property "Value" "10uF" (id 1) (at 415.29 313.6962 0)
+    (property "Value" "1uF" (id 1) (at 415.29 313.6962 0)
       (effects (font (size 1.27 1.27)) (justify left))
     )
@@
       (effects (font (size 1.27 1.27)) (justify left))
     )
-    (property "Value" "10uF" (id 1) (at 372.11 229.8762 0)
+    (property "Value" "1uF" (id 1) (at 372.11 229.8762 0)
       (effects (font (size 1.27 1.27)) (justify left))
     )
@@
     )
     (path "/cb051840-dec9-4514-9b7f-4aac00c0f4e6"
-      (reference "C9") (unit 1) (value "10uF") (footprint "Capacitor_SMD:C_0603_1608Metric")
+      (reference "C9") (unit 1) (value "1uF") (footprint "Capacitor_SMD:C_0603_1608Metric")
     )
     (path "/20eac1c0-0b1b-4873-b7c1-92ab058ded19"
@@
     )
     (path "/27dd96c9-b427-47cd-a438-de737beeeafd"
-      (reference "C11") (unit 1) (value "10uF") (footprint "Capacitor_SMD:C_0603_1608Metric")
+      (reference "C11") (unit 1) (value "1uF") (footprint "Capacitor_SMD:C_0603_1608Metric")
     )
     (path "/b85d1bc8-1cee-4f8a-bf1f-061ae3c4ebeb"
